Commit message: few changes

File: ninni_robot_arm/urdf/ninni_robot_arm.urdf (robot description, URDF)
Before this commit: robot ninni_robot_arm, 4 links, 3 joints
Links:
- added link gripper_link; visual box size=0.04 0.02 0.04
- added link link4; visual box size=0.03 0.03 0.08
- added link link5; visual cylinder length=0.06 radius=0.02
Joints:
- added joint gripper_joint: type fixed, parent link5, child gripper_link, origin xyz=0 0 0.06 rpy=0 0 0
- added joint joint4: type revolute, parent link3, child link4, origin xyz=0 0 0.12 rpy=0 0 0, axis 0 1 0, limit lower=-1.57 upper=1.57 effort=10 velocity=1.0
- added joint joint5: type revolute, parent link4, child link5, origin xyz=0 0 0.08 rpy=0 0 0, axis 0 0 1, limit lower=-3.14 upper=3.14 effort=10 velocity=1.0
- joint joint2: origin xyz=0 0 0.15 rpy=0 1.57 0 -> xyz=0 0 0.15 rpy=0 0 0
