Commit message: ADD : config and moveit

File: ninni_robot_arm/urdf/ninni_arm.urdf (robot description, URDF)
Before this commit: robot onshape_export, 5 links, 4 joints
Links:
- link base_of_shoulder: geometry collision mesh filename=package://ninni_robot_arm/meshes/base_of_shoulder.stl; collision mesh filename=package://ninni_robot_arm/meshes/j2_servo.stl
- link base_servo_board: geometry collision mesh filename=package://ninni_robot_arm/meshes/base_servo_board.stl; collision mesh filename=package://ninni_robot_arm/meshes/servo_motor_sts3215_v10.stl
- link left_cover: geometry collision mesh filename=package://ninni_robot_arm/meshes/elbow_left.stl; collision mesh filename=package://ninni_robot_arm/meshes/elbow_right.stl
- link left_cover_2: geometry collision mesh filename=package://ninni_robot_arm/meshes/left_cover__2.stl; collision mesh filename=package://ninni_robot_arm/meshes/left_cover__3.stl
- link shoulder_left: geometry collision mesh filename=package://ninni_robot_arm/meshes/j3_servo.stl; collision mesh filename=package://ninni_robot_arm/meshes/left_cover.stl
Joints:
- joint Servor_1_to_waist: limit lower=-12.5664 upper=0 effort=10 velocity=10 -> lower=-6.28319 upper=6.28319 effort=10 velocity=10
- joint left_1_arm: limit lower=-1.65806 upper=1.65806 effort=10 velocity=10 -> lower=-1.5708 upper=1.5708 effort=10 velocity=10; origin xyz=-0.0303266 0.021403 0.0916284 rpy=1.5708 0 1.5708 -> xyz=0.000373062 -0.0169731 0.049 rpy=1.5708 -0 -3.14159; parent base_of_shoulder -> base_servo_board
- joint left_2_arm: limit lower=-2.26893 upper=2.26893 effort=10 velocity=10 -> lower=-2.0944 upper=2.0944 effort=10 velocity=10; origin xyz=-0 0.096 -1.91259e-05 rpy=-0 -0 -0 -> xyz=0 0.096 -1.91259e-05 rpy=0 -0 0

File: onshape_export/robot_old.urdf (robot description, URDF)
Before this commit: robot onshape_export, 5 links, 4 joints
Joints:
- joint Servor_1_to_waist: limit lower=-12.5664 upper=0 effort=10 velocity=10 -> lower=-3.14159 upper=3.14159 effort=10 velocity=10
- joint left_1_arm: limit lower=-1.65806 upper=1.65806 effort=10 velocity=10 -> lower=-1.5708 upper=1.5708 effort=10 velocity=10
- joint left_2_arm: limit lower=-2.26893 upper=2.26893 effort=10 velocity=10 -> lower=-2.0944 upper=2.0944 effort=10 velocity=10; origin xyz=-0 0.096 -1.91259e-05 rpy=-0 -0 -0 -> xyz=0 0.096 -1.91259e-05 rpy=0 -0 0
