Commit message: ADD : adding animation plan by code another python file top re order of sequence of chain and joint that I set up eariler in moveit assistant.

File: ninni_arm_moveit_config/config/onshape_export.ros2_control.xacro (robot description, xacro)
@@ -8,4 +8,11 @@
                 <plugin>mock_components/GenericSystem</plugin>
             </hardware>
+            <joint name="Servor_1_to_waist">
+                <command_interface name="position"/>
+                <state_interface name="position">
+                  <param name="initial_value">${initial_positions['Servor_1_to_waist']}</param>
+                </state_interface>
+                <state_interface name="velocity"/>
+            </joint>
             <joint name="left_1_arm">
                 <command_interface name="position"/>
@@ -29,11 +36,4 @@
                 <state_interface name="velocity"/>
             </joint>
-            <joint name="Servor_1_to_waist">
-                <command_interface name="position"/>
-                <state_interface name="position">
-                  <param name="initial_value">${initial_positions['Servor_1_to_waist']}</param>
-                </state_interface>
-                <state_interface name="velocity"/>
-            </joint>
         </ros2_control>
     </xacro:macro>

File: ninni_robot_arm/urdf/ninni_arm.urdf (robot description, URDF)
Before this commit: robot onshape_export, 5 links, 4 joints
Links:
- link base_of_shoulder: mass 0 -> 0.158649
- link base_servo_board: mass 0 -> 0.129831
- link left_cover: mass 0 -> 0.0917628
- link left_cover_2: mass 0 -> 0.0268203; geometry collision mesh filename=package://ninni_robot_arm/meshes/left_cover__2.stl; collision mesh filename=package://ninni_robot_arm/meshes/left_cover__3.stl
- link shoulder_left: mass 0 -> 0.0926197
Joints:
- joint Servor_1_to_waist: child base_servo_board -> base_of_shoulder; limit lower=-6.28319 upper=6.28319 effort=10 velocity=10 -> lower=-3.14159 upper=3.14159 effort=10 velocity=10; origin xyz=-0.0133535 0.021776 0.0426284 rpy=0 -0 -1.5708 -> xyz=-0.0133535 0.021776 0.0426284 rpy=-3.14159 0 -1.5708; parent base_of_shoulder -> base_servo_board
- joint left_1_arm: origin xyz=0.000373062 -0.0169731 0.049 rpy=1.5708 -0 -3.14159 -> xyz=0.000373 0.0169731 -0.049 rpy=-1.5708 -0 -3.14159; parent base_servo_board -> base_of_shoulder

File: onshape_export/robot.urdf (robot description, URDF)
Before this commit: robot onshape_export, 5 links, 4 joints
Links:
- link base_of_shoulder: mass 0 -> 0.158649
- link base_servo_board: mass 0 -> 0.129831
- link left_cover: mass 0 -> 0.0917628
- link left_cover_2: mass 0 -> 0.0268203; geometry collision mesh filename=package://assets/left_cover__2.stl; collision mesh filename=package://assets/left_cover__3.stl
- link shoulder_left: mass 0 -> 0.0926197
Joints:
- joint Servor_1_to_waist: child base_servo_board -> base_of_shoulder; origin xyz=-0.0133535 0.021776 0.0426284 rpy=0 -0 -1.5708 -> xyz=-0.0133535 0.021776 0.0426284 rpy=-3.14159 0 -1.5708; parent base_of_shoulder -> base_servo_board
- joint left_1_arm: origin xyz=-0.0303266 0.021403 0.0916284 rpy=1.5708 0 1.5708 -> xyz=0.000373 0.0169731 -0.049 rpy=-1.5708 -0 -3.14159

File: onshape_export/robot_view_new.urdf (robot description, URDF)
Before this commit: robot onshape_export, 5 links, 4 joints
Links:
- link base_of_shoulder: mass 0 -> 0.158649
- link base_servo_board: mass 0 -> 0.129831
- link left_cover: mass 0 -> 0.0917628
- link left_cover_2: mass 0 -> 0.0268203; geometry collision mesh filename=file:///home/ninnin/Ninni_Robot_Arm/onshape_export/assets/l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; collision mesh filename=file:///home/ninnin/Ninni_Robot_Arm/onshape_export/assets/l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
- link shoulder_left: mass 0 -> 0.0926197
Joints:
- joint Servor_1_to_waist: child base_servo_board -> base_of_shoulder; limit lower=-12.5664 upper=0 effort=10 velocity=10 -> lower=-3.14159 upper=3.14159 effort=10 velocity=10; origin xyz=-0.0133535 0.021776 0.0426284 rpy=0 -0 -1.5708 -> xyz=-0.0133535 0.021776 0.0426284 rpy=-3.14159 0 -1.5708; parent base_of_shoulder -> base_servo_board
- joint left_1_arm: limit lower=-0.906676 upper=2.1651 effort=10 velocity=10 -> lower=-1.5708 upper=1.5708 effort=10 velocity=10; origin xyz=-0.0303266 0.021403 0.0916284 rpy=1.5708 0.629214 1.5708 -> xyz=0.000373 0.0169731 -0.049 rpy=-1.5708 -0 -3.14159
- joint left_2_arm: limit lower=-1.97473 upper=2.21406 effort=10 velocity=10 -> lower=-2.0944 upper=2.0944 effort=10 velocity=10; origin xyz=-0 0.096 -1.91259e-05 rpy=0 0 -0.119662 -> xyz=0 0.096 -1.91259e-05 rpy=0 -0 0
- joint left_3_arm: limit lower=-2.65749 upper=1.5313 effort=10 velocity=10 -> lower=-2.0944 upper=2.0944 effort=10 velocity=10; origin xyz=-0 0.096 -1.91259e-05 rpy=-0 0 0.563091 -> xyz=0 0.096 -1.91259e-05 rpy=0 0 0
